File: watch/LED_Driver.sch (KiCad schematic (older format))
At the start: 80 parts, among them IC1 IS32FL3237-TQLA3-TR

Commit message: V2 after Feedback
Changed lines of the file:
@@
 L power:GND #PWR0110
 U 1 1 619ACD04
-P 4150 5800
-F 0 "#PWR0110" H 4150 5550 50  0001 C CNN
-F 1 "GND" V 4155 5672 50  0000 R CNN
-F 2 "" H 4150 5800 50  0001 C CNN
-F 3 "" H 4150 5800 50  0001 C CNN
-	1    4150 5800
-	0    1    1    0
+P 3950 6000
+F 0 "#PWR0110" H 3950 5750 50  0001 C CNN
+F 1 "GND" V 3955 5872 50  0000 R CNN
+F 2 "" H 3950 6000 50  0001 C CNN
+F 3 "" H 3950 6000 50  0001 C CNN
+	1    3950 6000
+	1    0    0    -1
 $EndComp
 Wire Wire Line
@@
 L power:GND #PWR0111
 U 1 1 619B02F8
-P 6350 4100
-F 0 "#PWR0111" H 6350 3850 50  0001 C CNN
-F 1 "GND" H 6355 3927 50  0000 C CNN
-F 2 "" H 6350 4100 50  0001 C CNN
-F 3 "" H 6350 4100 50  0001 C CNN
-	1    6350 4100
-	0    -1   -1   0
+P 6350 4500
+F 0 "#PWR0111" H 6350 4250 50  0001 C CNN
+F 1 "GND" H 6355 4327 50  0000 C CNN
+F 2 "" H 6350 4500 50  0001 C CNN
+F 3 "" H 6350 4500 50  0001 C CNN
+	1    6350 4500
+	1    0    0    -1
 $EndComp
 Wire Wire Line
 	4300 4100 3500 4100
-$Comp
-L power:GND #PWR0112
-U 1 1 619B15BE
-P 3500 4100
-F 0 "#PWR0112" H 3500 3850 50  0001 C CNN
-F 1 "GND" H 3505 3927 50  0000 C CNN
-F 2 "" H 3500 4100 50  0001 C CNN
-F 3 "" H 3500 4100 50  0001 C CNN
-	1    3500 4100
-	0    1    1    0
-$EndComp
 Wire Wire Line
 	5200 2350 5300 2350
 Wire Wire Line
 	5300 2350 5300 2500
-Connection ~ 5300 2350
 $Comp
 L power:GND #PWR0113
 U 1 1 619B2D1B
-P 5300 2250
-F 0 "#PWR0113" H 5300 2000 50  0001 C CNN
-F 1 "GND" V 5305 2122 50  0000 R CNN
-F 2 "" H 5300 2250 50  0001 C CNN
-F 3 "" H 5300 2250 50  0001 C CNN
-	1    5300 2250
-	-1   0    0    1
+P 4250 2450
+F 0 "#PWR0113" H 4250 2200 50  0001 C CNN
+F 1 "GND" V 4255 2322 50  0000 R CNN
+F 2 "" H 4250 2450 50  0001 C CNN
+F 3 "" H 4250 2450 50  0001 C CNN
+	1    4250 2450
+	1    0    0    -1
 $EndComp
 $Comp
@@
 L power:GND #PWR0114
 U 1 1 619B9712
-P 5400 6300
-F 0 "#PWR0114" H 5400 6050 50  0001 C CNN
-F 1 "GND" H 5405 6127 50  0000 C CNN
-F 2 "" H 5400 6300 50  0001 C CNN
-F 3 "" H 5400 6300 50  0001 C CNN
-	1    5400 6300
-	0    -1   -1   0
-$EndComp
-Connection ~ 5400 6300
+P 5600 6900
+F 0 "#PWR0114" H 5600 6650 50  0001 C CNN
+F 1 "GND" H 5605 6727 50  0000 C CNN
+F 2 "" H 5600 6900 50  0001 C CNN
+F 3 "" H 5600 6900 50  0001 C CNN
+	1    5600 6900
+	1    0    0    -1
+$EndComp
 Wire Wire Line
 	5000 6300 5100 6300
@@
 	4800 6300 4800 6800
 Wire Wire Line
-	4500 6300 4400 6300
-Wire Wire Line
-	4400 6300 4400 6800
-Wire Wire Line
-	4400 6800 4500 6800
-$Comp
-L power:GND #PWR0115
-U 1 1 619C0D07
-P 4400 6300
-F 0 "#PWR0115" H 4400 6050 50  0001 C CNN
-F 1 "GND" H 4405 6127 50  0000 C CNN
-F 2 "" H 4400 6300 50  0001 C CNN
-F 3 "" H 4400 6300 50  0001 C CNN
-	1    4400 6300
-	0    1    1    0
-$EndComp
-Connection ~ 4400 6300
-Wire Wire Line
-	4350 5800 4150 5800
-Connection ~ 4350 5800
+	3950 5800 3950 6000
 Wire Wire Line
 	5400 5200 5400 6050
@@
 	6100 4100 6350 4100
 Wire Wire Line
-	5300 2350 5300 2250
-Wire Wire Line
 	5800 5200 5800 5700
-Wire Wire Line
-	5800 5700 6100 5700
 $Comp
 L power:GND #PWR05
 U 1 1 61B50786
-P 6100 5700
-F 0 "#PWR05" H 6100 5450 50  0001 C CNN
-F 1 "GND" V 6105 5572 50  0000 R CNN
-F 2 "" H 6100 5700 50  0001 C CNN
-F 3 "" H 6100 5700 50  0001 C CNN
-	1    6100 5700
-	0    -1   -1   0
+P 5800 5700
+F 0 "#PWR05" H 5800 5450 50  0001 C CNN
+F 1 "GND" V 5805 5572 50  0000 R CNN
+F 2 "" H 5800 5700 50  0001 C CNN
+F 3 "" H 5800 5700 50  0001 C CNN
+	1    5800 5700
+	1    0    0    -1
 $EndComp
 Text Label 4000 650  0    50   ~ 0
@@
 Wire Wire Line
 	3800 3300 3800 1350
+Wire Wire Line
+	4350 5800 3950 5800
+Connection ~ 4350 5800
+Wire Wire Line
+	4400 6800 4500 6800
+Wire Wire Line
+	4400 6300 4400 6800
+Wire Wire Line
+	4500 6300 4400 6300
+Wire Wire Line
+	4400 6800 3950 6800
+Wire Wire Line
+	3950 6800 3950 6950
+Connection ~ 4400 6800
+$Comp
+L power:GND #PWR?
+U 1 1 61B465E8
+P 3950 6950
+F 0 "#PWR?" H 3950 6700 50  0001 C CNN
+F 1 "GND" H 3955 6777 50  0000 C CNN
+F 2 "" H 3950 6950 50  0001 C CNN
+F 3 "" H 3950 6950 50  0001 C CNN
+	1    3950 6950
+	1    0    0    -1
+$EndComp
+Wire Wire Line
+	5400 6800 5600 6800
+Wire Wire Line
+	5600 6800 5600 6900
+Connection ~ 5400 6800
+Wire Wire Line
+	6350 4100 6350 4500
+$Comp
+L power:GND #PWR?
+U 1 1 61BBB01C
+P 3500 4500
+F 0 "#PWR?" H 3500 4250 50  0001 C CNN
+F 1 "GND" H 3505 4327 50  0000 C CNN
+F 2 "" H 3500 4500 50  0001 C CNN
+F 3 "" H 3500 4500 50  0001 C CNN
+	1    3500 4500
+	1    0    0    -1
+$EndComp
+Wire Wire Line
+	3500 4100 3500 4500
+Wire Wire Line
+	5200 2350 4250 2350
+Wire Wire Line
+	4250 2350 4250 2450
+Connection ~ 5200 2350
 $EndSCHEMATC
