File: watch/watch.sch (KiCad schematic (older format))
At the start: 22 parts, among them SW1 ButtonWakeup, U1 STM32L031F4Px, Y1 CR_32kHz

Commit message: no more vias below metallic components; cleaned up some tracks
Parts:
- removed TP6: TP_GND, TestPoint:TestPoint_Pad_D1.0mm, symbol Connector:TestPoint
- removed TP7: TP_3V3, TestPoint:TestPoint_Pad_D1.0mm, symbol Connector:TestPoint
Changed lines of the file:
@@
-$EndComp
-Wire Wire Line
-	7700 1900 7700 1750
-Connection ~ 7700 1900
-Wire Wire Line
-	7700 2300 7700 2450
-Connection ~ 7700 2300
-$Comp
-L Connector:TestPoint TP6
-U 1 1 619CABCC
-P 7700 1750
-F 0 "TP6" H 7758 1868 50  0000 L CNN
-F 1 "TP_GND" H 7758 1777 50  0000 L CNN
-F 2 "TestPoint:TestPoint_Pad_D1.0mm" H 7900 1750 50  0001 C CNN
-F 3 "~" H 7900 1750 50  0001 C CNN
-	1    7700 1750
-	1    0    0    -1
-$EndComp
-$Comp
-L Connector:TestPoint TP7
-U 1 1 619CFA24
-P 7700 2450
-F 0 "TP7" H 7642 2476 50  0000 R CNN
-F 1 "TP_3V3" H 7642 2567 50  0000 R CNN
-F 2 "TestPoint:TestPoint_Pad_D1.0mm" H 7900 2450 50  0001 C CNN
-F 3 "~" H 7900 2450 50  0001 C CNN
-	1    7700 2450
-	-1   0    0    1
 $EndComp
 Wire Wire Line

Commit message: V2 after Feedback
Parts:
- added TP6: UART_TX, TestPoint:TestPoint_Pad_D1.0mm, symbol Connector:TestPoint
- added TP7: UART_RX, TestPoint:TestPoint_Pad_D1.0mm, symbol Connector:TestPoint
Connections:
- net at U1.8 (PA2): now also TP6.1
- net at U1.9 (PA3): now also TP7.1
- no-connect marks 7 -> 5
Other:
- moved on the sheet: BT1, C1, C5, C6, C7, R4, R51, SW1
