File: watch/LED_Driver.kicad_sch (KiCad schematic)
At the start: 69 parts, among them IC1 IS32FL3237-TQLA3-TR, IC2 TMUX1237DCKR

Commit message: as ordered V1.4
Parts:
- removed C2: 100nF, custom:C_0603_1608Metric, symbol Device:C_Small
- removed IC1: IS32FL3237-TQLA3-TR, SamacSys_Parts:QFP50P900X900X120-49N, symbol IS32FL3237:IS32FL3237-TQLA3-TR
- removed R28, R31: 2k, custom:R_0603_1608Metric, symbol Device:R_Small
- added IC1: IS32FL3237-TQLA3-TR, SamacSys_Parts:QFP50P900X900X120-49N, symbol SamacSys_Parts:IS32FL3237-TQLA3-TR
- added R7: 10k, custom:R_0603_1608Metric, symbol Device:R_Small
Connections:
- net +3V3 is gone; now on net VCC: IC2.2 (VDD), IC2.4 (D)
- net LED_BANK: now also R7.2; no longer IC2.6 (SEL)
- net SCL: now also IC1.46 (SCL)
- net SDA: now also IC1.45 (SDA)
- net VCC: now also R20.2, IC1.41 (VCC)
- net at D57.1 (K), D58.1 (K): now also IC1.10 (OUT11)
- net at D59.1 (K), D60.1 (K): now also IC1.11 (OUT12)
- net at D1.1 (K), D2.1 (K): now also IC1.12 (OUT13)
- net at D3.1 (K), D4.1 (K): now also IC1.13 (OUT14)
- net at D5.1 (K), D6.1 (K): now also IC1.14 (OUT15)
- net at D7.1 (K), D8.1 (K): now also IC1.15 (OUT16)
- net at D10.1 (K), D9.1 (K): now also IC1.16 (OUT17)
- net at D11.1 (K), D12.1 (K): now also IC1.17 (OUT18)
- net at D13.1 (K), D14.1 (K): now also IC1.20 (OUT19)
- net at D15.1 (K), D16.1 (K): now also IC1.21 (OUT20)
- net at D17.1 (K), D18.1 (K): now also IC1.22 (OUT21)
- net at D19.1 (K), D20.1 (K): now also IC1.23 (OUT22)
- net at D21.1 (K), D22.1 (K): now also IC1.24 (OUT23_1)
- net at D23.1 (K), D24.1 (K): now also IC1.25 (OUT24)
- net at D25.1 (K), D26.1 (K): now also IC1.26 (OUT25)
- net at D27.1 (K), D28.1 (K): now also IC1.27 (OUT26)
- net at D29.1 (K), D30.1 (K): now also IC1.28 (OUT27)
- net at D31.1 (K), D32.1 (K): now also IC1.29 (OUT28)
- net at D45.1 (K), D46.1 (K): now also IC1.3 (OUT5)
- net at D33.1 (K), D34.1 (K): now also IC1.30 (OUT29)
- net at D35.1 (K), D36.1 (K): now also IC1.31 (OUT30)
- net at D37.1 (K), D38.1 (K): now also IC1.32 (OUT31)
- net at D39.1 (K), D40.1 (K): now also IC1.34 (OUT32)
- net at D41.1 (K), D42.1 (K): now also IC1.35 (OUT33)
- net at D43.1 (K), D44.1 (K): now also IC1.36 (OUT34)
- net at R24.2: now also IC1.44 (ISET)
- net at D47.1 (K), D48.1 (K): now also IC1.5 (OUT6)
- net at D49.1 (K), D50.1 (K): now also IC1.6 (OUT7)
- net at D51.1 (K), D52.1 (K): now also IC1.7 (OUT8)
- net at D53.1 (K), D54.1 (K): now also IC1.8 (OUT9)
- net at D55.1 (K), D56.1 (K): now also IC1.9 (OUT10)
- net EN: no longer names the net of R20.1
- net EN: now also IC1.39 (SDB)
- net GND renamed GND1
- net GND1: now also IC1.18 (GND_2), IC1.19 (GND_3), IC1.33 (GND_4), IC1.4 (GND_1), IC1.40 (AD), IC1.42 (GND_5), IC1.43 (GND_6), IC1.49 (OUT23_2); no longer R20.2
- new net: IC2.6 (SEL), R7.1
Other:
- moved on the sheet: R20
