File: watch/watch.kicad_sch (KiCad schematic)
At the start: 92 parts, among them Q1 Q_NMOS_GSD, Q2 Q_NMOS_GSD, Q3 Q_NMOS_GSD, Q4 Q_NMOS_GSD, U1 STM32L071CBTx, Y1 Crystal

Commit message: added unfinished footprint for DFN0606 FETs
Parts:
- Q1, Q2, Q3, Q4: value Q_NMOS_GSD -> DMN2991UFZ
Changed lines of the file:
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@@
 			)
 		)
-		(property "Value" "Q_NMOS_GSD"
+		(property "Value" "DMN2991UFZ"
 			(at 445.77 325.12 0)
 			(effects
@@
 			)
 		)
-		(property "Value" "Q_NMOS_GSD"
+		(property "Value" "DMN2991UFZ"
 			(at 481.33 325.12 0)
 			(effects
@@
 			)
 		)
-		(property "Value" "Q_NMOS_GSD"
+		(property "Value" "DMN2991UFZ"
 			(at 408.94 325.12 0)
 			(effects
@@
 			)
 		)
-		(property "Value" "Q_NMOS_GSD"
+		(property "Value" "DMN2991UFZ"
 			(at 373.38 325.12 0)
 			(effects

Commit message: added DFN0606 footprint
Parts:
- Q1, Q2, Q3, Q4: footprint Package_TO_SOT_SMD:SOT-23 -> DFN0603:DFN0606
Changed lines of the file:
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@@
 			)
 		)
-		(property "Footprint" "Package_TO_SOT_SMD:SOT-23"
+		(property "Footprint" "DFN0603:DFN0606"
 			(at 444.5 317.5 0)
 			(effects
@@
 			)
 		)
-		(property "Footprint" "Package_TO_SOT_SMD:SOT-23"
+		(property "Footprint" "DFN0603:DFN0606"
 			(at 480.06 317.5 0)
 			(effects
@@
 			)
 		)
-		(property "Footprint" "Package_TO_SOT_SMD:SOT-23"
+		(property "Footprint" "DFN0603:DFN0606"
 			(at 407.67 317.5 0)
 			(effects
@@
 			)
 		)
-		(property "Footprint" "Package_TO_SOT_SMD:SOT-23"
+		(property "Footprint" "DFN0603:DFN0606"
 			(at 372.11 317.5 0)
 			(effects

Commit message: removed low side FETs, started PCB
Parts:
- removed Q1, Q2, Q3, Q4: DMN2991UFZ, DFN0603:DFN0606, symbol Transistor_FET:Q_NMOS_GSD
- removed RN2: 1M, Resistor_SMD:R_Array_Concave_4x0402, symbol Device:R_Pack04
- removed RN3: 22, Resistor_SMD:R_Array_Concave_4x0402, symbol Device:R_Pack04
- D1, D10, D11, D12, D13, D14, D15, D16, D17, D18, D19, D2, D20, D21, D22, D23, D24, D25, D26, D27, D28, D29, D3, D30, D31, D32, D33, D34, D35, D36, D37, D38, D39, D4, D40, D41, D42, D43, D44, D45, D46, D47, D48, D49, D5, D50, D51, D52, D53, D54, D55, D56, D57, D58, D59, D6, D60, D7, D8, D9: footprint LED_SMD:LED_0402_1005Metric -> LED_Without_Dot:LED402_without_dot
- RN1: value 1k -> 100
- Y1: value Crystal -> 3131M-32.768DTTLRRL
Connections:
- net LED_SINK_ROW0_GPIO: now also RN1.4 (R4.1)
- net LED_SINK_ROW1_GPIO: now also RN1.3 (R3.1)
- net LED_SINK_ROW2_GPIO: now also RN1.2 (R2.1)
- net LED_SINK_ROW3_GPIO: now also RN1.1 (R1.1)
- net LED_SOURCE_COLUMN0: now also D2.2 (A), D3.2 (A), D4.2 (A); no longer D16.2 (A), D31.2 (A), D46.2 (A)
- net LED_SOURCE_COLUMN1: now also D5.2 (A), D6.2 (A), D7.2 (A), D8.2 (A); no longer D17.2 (A), D2.2 (A), D32.2 (A), D47.2 (A)
- net LED_SOURCE_COLUMN10: now also D42.2 (A), D43.2 (A), D44.2 (A); no longer D11.2 (A), D26.2 (A), D56.2 (A)
- net LED_SOURCE_COLUMN11: now also D45.2 (A), D46.2 (A), D47.2 (A), D48.2 (A); no longer D12.2 (A), D27.2 (A), D42.2 (A), D57.2 (A)
- net LED_SOURCE_COLUMN12: now also D49.2 (A), D50.2 (A), D51.2 (A), D52.2 (A); no longer D13.2 (A), D28.2 (A), D43.2 (A), D58.2 (A)
- net LED_SOURCE_COLUMN13: now also D53.2 (A), D54.2 (A), D55.2 (A), D56.2 (A); no longer D14.2 (A), D29.2 (A), D44.2 (A), D59.2 (A)
- net LED_SOURCE_COLUMN14: now also D57.2 (A), D58.2 (A), D59.2 (A); no longer D15.2 (A), D30.2 (A), D45.2 (A)
- net LED_SOURCE_COLUMN2: now also D10.2 (A), D11.2 (A), D12.2 (A), D9.2 (A); no longer D18.2 (A), D3.2 (A), D33.2 (A), D48.2 (A)
- net LED_SOURCE_COLUMN3: now also D13.2 (A), D14.2 (A), D15.2 (A), D16.2 (A); no longer D19.2 (A), D34.2 (A), D4.2 (A), D49.2 (A)
- net LED_SOURCE_COLUMN4: now also D17.2 (A), D18.2 (A), D19.2 (A); no longer D35.2 (A), D5.2 (A), D50.2 (A)
- net LED_SOURCE_COLUMN5: now also D22.2 (A), D23.2 (A), D24.2 (A); no longer D36.2 (A), D51.2 (A), D6.2 (A)
- net LED_SOURCE_COLUMN6: now also D25.2 (A), D26.2 (A), D27.2 (A), D28.2 (A); no longer D22.2 (A), D37.2 (A), D52.2 (A), D7.2 (A)
- net LED_SOURCE_COLUMN7: now also D29.2 (A), D30.2 (A), D31.2 (A), D32.2 (A); no longer D23.2 (A), D38.2 (A), D53.2 (A), D8.2 (A)
- net LED_SOURCE_COLUMN8: now also D33.2 (A), D34.2 (A), D35.2 (A), D36.2 (A); no longer D24.2 (A), D39.2 (A), D54.2 (A), D9.2 (A)
- net LED_SOURCE_COLUMN9: now also D37.2 (A), D38.2 (A), D39.2 (A); no longer D10.2 (A), D25.2 (A), D55.2 (A)
- new net: D12.1 (K), D16.1 (K), D20.1 (K), D24.1 (K), D28.1 (K), D32.1 (K), D36.1 (K), D4.1 (K), D40.1 (K), D44.1 (K), D48.1 (K), D52.1 (K), D56.1 (K), D60.1 (K), D8.1 (K), RN1.8 (R1.2)
- new net: D1.1 (K), D13.1 (K), D17.1 (K), D21.1 (K), D25.1 (K), D29.1 (K), D33.1 (K), D37.1 (K), D41.1 (K), D45.1 (K), D49.1 (K), D5.1 (K), D53.1 (K), D57.1 (K), D9.1 (K), RN1.5 (R4.2)
- new net: D10.1 (K), D14.1 (K), D18.1 (K), D2.1 (K), D22.1 (K), D26.1 (K), D30.1 (K), D34.1 (K), D38.1 (K), D42.1 (K), D46.1 (K), D50.1 (K), D54.1 (K), D58.1 (K), D6.1 (K), RN1.6 (R3.2)
- new net: D11.1 (K), D15.1 (K), D19.1 (K), D23.1 (K), D27.1 (K), D3.1 (K), D31.1 (K), D35.1 (K), D39.1 (K), D43.1 (K), D47.1 (K), D51.1 (K), D55.1 (K), D59.1 (K), D7.1 (K), RN1.7 (R2.2)
Other:
- moved on the sheet: RN1

Commit message: V1.6 basic layout done
Parts:
- removed RN1: 100, Resistor_SMD:R_Array_Concave_4x0402, symbol Device:R_Pack04
- removed RN4: 22, Resistor_SMD:R_Array_Concave_4x0402, symbol Device:R_Pack04
- added R10, R8, R9: 22, Resistor_SMD:R_0603_1608Metric, symbol Device:R
- added R4, R5, R6, R7: 100, Resistor_SMD:R_0603_1608Metric, symbol Device:R
- C1, C10, C11, C12, C13, C2, C3, C4, C5, C7, C8, C9: footprint Capacitor_SMD:C_0402_1005Metric -> Capacitor_SMD:C_0603_1608Metric
- D1, D10, D11, D12, D13, D14, D15, D16, D17, D18, D19, D2, D20, D21, D22, D23, D24, D25, D26, D27, D28, D29, D3, D30, D31, D32, D33, D34, D35, D36, D37, D38, D39, D4, D40, D41, D42, D43, D44, D45, D46, D47, D48, D49, D5, D50, D51, D52, D53, D54, D55, D56, D57, D58, D59, D6, D60, D7, D8, D9: footprint LED_Without_Dot:LED402_without_dot -> LED_SMD:LED_0603_1608Metric
- R1, R2, R3: footprint Resistor_SMD:R_0402_1005Metric -> Resistor_SMD:R_0603_1608Metric
- TP1, TP2, TP3, TP4, TP5: footprint TestPoint:TestPoint_Pad_D1.0mm -> TestPoint:TestPoint_Pad_D2.0mm
Connections:
- net LED_SINK_ROW0_GPIO: now also R7.2
- net LED_SINK_ROW1_GPIO: now also R6.2
- net LED_SINK_ROW2_GPIO: now also R5.2
- net LED_SINK_ROW3_GPIO: now also R4.2
- net NRST: now also R10.1
- net SWCLK: now also R9.1
- net SWDIO: now also R8.1
- net VDD: now also TP1.1
- net at D12.1 (K), D16.1 (K), D20.1 (K)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: now also R4.1
- net at D1.1 (K), D13.1 (K), D17.1 (K)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: now also R7.1
- net at TP3.1: now also R9.2
- net at D10.1 (K), D14.1 (K), D18.1 (K)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: now also R6.1
- net at D11.1 (K), D15.1 (K), D19.1 (K)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: now also R5.1
- net at TP2.1: now also R8.2
- net at TP4.1: now also R10.2

Commit message: V1.6 done?
Parts:
- BT1: now not fitted
- C1, C10, C11, C2, C3, C4, C5, C9: LCSC Part # (none) -> C91183
- C12, C13: LCSC Part # (none) -> C86295
- C7, C8: LCSC Part # (none) -> C326779
- D1, D10, D11, D12, D13, D14, D15, D16, D17, D18, D19, D2, D20, D21, D22, D23, D24, D25, D26, D27, D28, D29, D3, D30, D31, D32, D33, D34, D35, D36, D37, D38, D39, D4, D40, D41, D42, D43, D44, D45, D46, D47, D48, D49, D5, D50, D51, D52, D53, D54, D55, D56, D57, D58, D59, D6, D60, D7, D8, D9: footprint LED_SMD:LED_0603_1608Metric -> LED_Without_Dot:0603; LCSC Part # (none) -> C284922
- R1, R2: LCSC Part # (none) -> C23162
- R10, R8, R9: LCSC Part # (none) -> C23345
- R3: LCSC Part # (none) -> C25805
- R4, R5, R6, R7: value 100 -> 160; LCSC Part # (none) -> C22814
- TP1, TP2, TP3, TP4, TP5: now not fitted; now left out of the parts list
- U1: LCSC Part # (none) -> C79758
- U2: value ~ -> BOSCH BMA400; LCSC Part # (none) -> C437655
- Y1: LCSC Part # (none) -> C42438016
Connections:
- net VDD: now also U1.17 (PA7), U2.10 (CSB); no longer U2.11 (PS)
