File: LED_Matrix.kicad_sch (KiCad schematic)
At the start: 68 parts, among them Q2 NPN, Q3 NPN, Q4 NPN, Q5 NPN

Commit message: V2 PCB first draft
Parts:
- removed D101, D105, D109, D113, D117, D61, D65, D69, D73, D77, D81, D85, D89, D93, D97: LED, symbol Device:LED
- removed Q2, Q3, Q4, Q5: NPN, symbol Simulation_SPICE:NPN
- added D1, D13, D17, D21, D25, D29, D33, D37, D41, D45, D49, D5, D53, D57, D9: LED, custom_lib:LED_0603_1608Metric_Pad1.05x0.95mm_HandSolder, symbol Device:LED
- added Q1, Q2, Q3, Q4: 2N7002H, Package_TO_SOT_SMD:SOT-23, symbol Transistor_FET:2N7002H
- added R10, R11, R12: 330/660, Resistor_SMD:R_0603_1608Metric_Pad0.98x0.95mm_HandSolder, symbol Device:R
- added R13, R14, R18, R19, R20: 10K, Resistor_SMD:R_0603_1608Metric_Pad0.98x0.95mm_HandSolder, symbol Device:R
- D10: renamed from D70; footprint (none) -> custom_lib:LED_0603_1608Metric_Pad1.05x0.95mm_HandSolder
- D11: renamed from D71; footprint (none) -> custom_lib:LED_0603_1608Metric_Pad1.05x0.95mm_HandSolder
- D12: renamed from D72; footprint (none) -> custom_lib:LED_0603_1608Metric_Pad1.05x0.95mm_HandSolder
- D14: renamed from D74; footprint (none) -> custom_lib:LED_0603_1608Metric_Pad1.05x0.95mm_HandSolder
- D15: renamed from D75; footprint (none) -> custom_lib:LED_0603_1608Metric_Pad1.05x0.95mm_HandSolder
- D16: renamed from D76; footprint (none) -> custom_lib:LED_0603_1608Metric_Pad1.05x0.95mm_HandSolder
- D18: renamed from D78; footprint (none) -> custom_lib:LED_0603_1608Metric_Pad1.05x0.95mm_HandSolder
- D19: renamed from D79; footprint (none) -> custom_lib:LED_0603_1608Metric_Pad1.05x0.95mm_HandSolder
- D2: renamed from D62; footprint (none) -> custom_lib:LED_0603_1608Metric_Pad1.05x0.95mm_HandSolder
- D20: renamed from D80; footprint (none) -> custom_lib:LED_0603_1608Metric_Pad1.05x0.95mm_HandSolder
- D22: renamed from D82; footprint (none) -> custom_lib:LED_0603_1608Metric_Pad1.05x0.95mm_HandSolder
- D23: renamed from D83; footprint (none) -> custom_lib:LED_0603_1608Metric_Pad1.05x0.95mm_HandSolder
- D24: renamed from D84; footprint (none) -> custom_lib:LED_0603_1608Metric_Pad1.05x0.95mm_HandSolder
- D26: renamed from D86; footprint (none) -> custom_lib:LED_0603_1608Metric_Pad1.05x0.95mm_HandSolder
- D27: renamed from D87; footprint (none) -> custom_lib:LED_0603_1608Metric_Pad1.05x0.95mm_HandSolder
- D28: renamed from D88; footprint (none) -> custom_lib:LED_0603_1608Metric_Pad1.05x0.95mm_HandSolder
- D3: renamed from D63; footprint (none) -> custom_lib:LED_0603_1608Metric_Pad1.05x0.95mm_HandSolder
- D30: renamed from D90; footprint (none) -> custom_lib:LED_0603_1608Metric_Pad1.05x0.95mm_HandSolder
- D31: renamed from D91; footprint (none) -> custom_lib:LED_0603_1608Metric_Pad1.05x0.95mm_HandSolder
- D32: renamed from D92; footprint (none) -> custom_lib:LED_0603_1608Metric_Pad1.05x0.95mm_HandSolder
- D34: renamed from D94; footprint (none) -> custom_lib:LED_0603_1608Metric_Pad1.05x0.95mm_HandSolder
- D35: renamed from D95; footprint (none) -> custom_lib:LED_0603_1608Metric_Pad1.05x0.95mm_HandSolder
- D36: renamed from D96; footprint (none) -> custom_lib:LED_0603_1608Metric_Pad1.05x0.95mm_HandSolder
- D38: renamed from D98; footprint (none) -> custom_lib:LED_0603_1608Metric_Pad1.05x0.95mm_HandSolder
- D39: renamed from D99; footprint (none) -> custom_lib:LED_0603_1608Metric_Pad1.05x0.95mm_HandSolder
- D4: renamed from D64; footprint (none) -> custom_lib:LED_0603_1608Metric_Pad1.05x0.95mm_HandSolder
- D40: renamed from D100; footprint (none) -> custom_lib:LED_0603_1608Metric_Pad1.05x0.95mm_HandSolder
- D42: renamed from D102; footprint (none) -> custom_lib:LED_0603_1608Metric_Pad1.05x0.95mm_HandSolder
- D43: renamed from D103; footprint (none) -> custom_lib:LED_0603_1608Metric_Pad1.05x0.95mm_HandSolder
- D44: renamed from D104; footprint (none) -> custom_lib:LED_0603_1608Metric_Pad1.05x0.95mm_HandSolder
- D46: renamed from D106; footprint (none) -> custom_lib:LED_0603_1608Metric_Pad1.05x0.95mm_HandSolder
- D47: renamed from D107; footprint (none) -> custom_lib:LED_0603_1608Metric_Pad1.05x0.95mm_HandSolder
- D48: renamed from D108; footprint (none) -> custom_lib:LED_0603_1608Metric_Pad1.05x0.95mm_HandSolder
- D50: renamed from D110; footprint (none) -> custom_lib:LED_0603_1608Metric_Pad1.05x0.95mm_HandSolder
- D51: renamed from D111; footprint (none) -> custom_lib:LED_0603_1608Metric_Pad1.05x0.95mm_HandSolder
- D52: renamed from D112; footprint (none) -> custom_lib:LED_0603_1608Metric_Pad1.05x0.95mm_HandSolder
- D54: renamed from D114; footprint (none) -> custom_lib:LED_0603_1608Metric_Pad1.05x0.95mm_HandSolder
- D55: renamed from D115; footprint (none) -> custom_lib:LED_0603_1608Metric_Pad1.05x0.95mm_HandSolder
- D56: renamed from D116; footprint (none) -> custom_lib:LED_0603_1608Metric_Pad1.05x0.95mm_HandSolder
- D58: renamed from D118; footprint (none) -> custom_lib:LED_0603_1608Metric_Pad1.05x0.95mm_HandSolder
- D59: renamed from D119; footprint (none) -> custom_lib:LED_0603_1608Metric_Pad1.05x0.95mm_HandSolder
- D6: renamed from D66; footprint (none) -> custom_lib:LED_0603_1608Metric_Pad1.05x0.95mm_HandSolder
- D60: renamed from D120; footprint (none) -> custom_lib:LED_0603_1608Metric_Pad1.05x0.95mm_HandSolder
- D7: renamed from D67; footprint (none) -> custom_lib:LED_0603_1608Metric_Pad1.05x0.95mm_HandSolder
- D8: renamed from D68; footprint (none) -> custom_lib:LED_0603_1608Metric_Pad1.05x0.95mm_HandSolder
- R15, R16, R17: value R -> 10K; footprint (none) -> Resistor_SMD:R_0603_1608Metric_Pad0.98x0.95mm_HandSolder
- R9: renamed from R14; value R -> 330/660; footprint (none) -> Resistor_SMD:R_0603_1608Metric_Pad0.98x0.95mm_HandSolder
Connections:
- net GND: now also R15.2, R16.2, Q1.2 (S), Q2.2 (S), Q3.2 (S), Q4.2 (S), R13.2, R14.2
- net LEDCOL0: now also D1.2 (A)
- net LEDCOL1: now also D5.2 (A)
- net LEDCOL10: now also D41.2 (A)
- net LEDCOL11: now also D45.2 (A)
- net LEDCOL12: now also D49.2 (A)
- net LEDCOL13: now also D53.2 (A)
- net LEDCOL14: now also D57.2 (A)
- net LEDCOL2: now also D9.2 (A)
- net LEDCOL3: now also D13.2 (A)
- net LEDCOL4: now also D17.2 (A)
- net LEDCOL5: now also D21.2 (A)
- net LEDCOL6: now also D25.2 (A)
- net LEDCOL7: now also D29.2 (A)
- net LEDCOL8: now also D33.2 (A)
- net LEDCOL9: now also D37.2 (A)
- net LEDROW0: now also R17.2
- net LEDROW1: now also R18.2
- net LEDROW2: now also R19.2
- net LEDROW3: now also R20.2
- net at R15.1: now also Q3.1 (G), R19.1
- net at D10.1 (K), D14.1 (K), D18.1 (K)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: now also R10.2; no longer R15.2
- net at D12.1 (K), D16.1 (K), D20.1 (K)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: now also R12.2; no longer R17.2
- net at D11.1 (K), D15.1 (K), D19.1 (K)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: now also R11.2; no longer R16.2
- net at R9.2: now also D1.1 (K), D13.1 (K), D17.1 (K), D21.1 (K), D25.1 (K), D29.1 (K), D33.1 (K), D37.1 (K), D41.1 (K), D45.1 (K), D49.1 (K), D5.1 (K), D53.1 (K), D57.1 (K), D9.1 (K)
- net at R17.1: now also Q1.1 (G), R13.1
- net at R9.1: now also Q1.3 (D)
- net at R16.1: now also Q4.1 (G), R20.1
- new net: Q2.3 (D), R10.1
- new net: Q3.3 (D), R11.1
- new net: Q4.3 (D), R12.1
- new net: Q2.1 (G), R14.1, R18.1
Other:
- moved on the sheet: D10, D11, D12, D14, D15, D16, D18, D19, D2, D20, D22, D23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

Commit message: review
Parts:
- R10, R11, R12, R9: value 330/660 -> 47
- R13, R14, R15, R16: value 10K -> 1M
