File: accel.kicad_sch (KiCad schematic)
At the start: 7 parts

Commit message: V2 PCB first draft
Parts:
- C10: renamed from C3; footprint custom:C_0603_1608Metric -> Capacitor_SMD:C_0603_1608Metric
- C8: renamed from C1; footprint custom:C_0603_1608Metric -> Capacitor_SMD:C_0603_1608Metric
- C9: renamed from C2; footprint custom:C_0603_1608Metric -> Capacitor_SMD:C_0603_1608Metric
- R6: renamed from R2; footprint custom:R_0603_1608Metric -> Resistor_SMD:R_0603_1608Metric_Pad0.98x0.95mm_HandSolder
- R7: renamed from R3; footprint custom:R_0603_1608Metric -> Resistor_SMD:R_0603_1608Metric_Pad0.98x0.95mm_HandSolder
- R8: renamed from R1; footprint custom:R_0603_1608Metric -> Resistor_SMD:R_0603_1608Metric_Pad0.98x0.95mm_HandSolder
- renumbered U1 to U2
Changed lines of the file:
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@@
 		(dnp no)
 		(fields_autoplaced yes)
-		(property "Reference" "#PWR01"
+		(property "Reference" "#PWR012"
 			(at 143.51 67.31 0)
 			(effects
@@
 			(project "watch"
 				(path "/71c31975-2c45-4d18-a25a-18e07a55d11e/53708456-0ae3-4e95-bf36-829cd83d6b3b"
-					(reference "#PWR01")
+					(reference "#PWR012")
 					(unit 1)
 				)
@@
 		(dnp no)
 		(fields_autoplaced yes)
-		(property "Reference" "#PWR03"
+		(property "Reference" "#PWR014"
 			(at 179.07 52.07 0)
 			(effects
@@
 			(project "watch"
 				(path "/71c31975-2c45-4d18-a25a-18e07a55d11e/53708456-0ae3-4e95-bf36-829cd83d6b3b"
-					(reference "#PWR03")
+					(reference "#PWR014")
 					(unit 1)
 				)
@@
 		(on_board yes)
 		(dnp no)
-		(property "Reference" "#PWR02"
+		(property "Reference" "#PWR013"
 			(at 143.51 97.79 0)
 			(effects
@@
 			(project "watch"
 				(path "/71c31975-2c45-4d18-a25a-18e07a55d11e/53708456-0ae3-4e95-bf36-829cd83d6b3b"
-					(reference "#PWR02")
+					(reference "#PWR013")
 					(unit 1)
 				)
@@
 		(on_board yes)
 		(dnp no)
-		(property "Reference" "C2"
+		(property "Reference" "C9"
 			(at 122.1232 68.6816 0)
 			(effects
@@
 			)
 		)
-		(property "Footprint" "custom:C_0603_1608Metric"
+		(property "Footprint" "Capacitor_SMD:C_0603_1608Metric"
 			(at 124.46 69.85 0)
 			(effects
@@
 			(project "watch"
 				(path "/71c31975-2c45-4d18-a25a-18e07a55d11e/53708456-0ae3-4e95-bf36-829cd83d6b3b"
-					(reference "C2")
+					(reference "C9")
 					(unit 1)
 				)
@@
 		(on_board yes)
 		(dnp no)
-		(property "Reference" "C3"
+		(property "Reference" "C10"
 			(at 132.2832 68.6816 0)
 			(effects
@@
 			)
 		)
-		(property "Footprint" "custom:C_0603_1608Metric"
+		(property "Footprint" "Capacitor_SMD:C_0603_1608Metric"
 			(at 134.62 69.85 0)
 			(effects
@@
 			(project "watch"
 				(path "/71c31975-2c45-4d18-a25a-18e07a55d11e/53708456-0ae3-4e95-bf36-829cd83d6b3b"
-					(reference "C3")
+					(reference "C10")
 					(unit 1)
 				)
@@
 		(on_board yes)
 		(dnp no)
-		(property "Reference" "R2"
+		(property "Reference" "R6"
 			(at 177.8 55.88 0)
 			(effects
@@
 			)
 		)
-		(property "Footprint" "custom:R_0603_1608Metric"
+		(property "Footprint" "Resistor_SMD:R_0603_1608Metric_Pad0.98x0.95mm_HandSolder"
 			(at 173.99 54.61 0)
 			(effects
@@
 			(project "watch"
 				(path "/71c31975-2c45-4d18-a25a-18e07a55d11e/53708456-0ae3-4e95-bf36-829cd83d6b3b"
-					(reference "R2")
+					(reference "R6")
 					(unit 1)
 				)
@@
 		(dnp no)
 		(fields_autoplaced yes)
-		(property "Reference" "U1"
+		(property "Reference" "U2"
 			(at 163.4841 54.61 0)
 			(effects
@@
 			(project "watch"
 				(path "/71c31975-2c45-4d18-a25a-18e07a55d11e/53708456-0ae3-4e95-bf36-829cd83d6b3b"
-					(reference "U1")
+					(reference "U2")
 					(unit 1)
 				)
@@
 		(on_board yes)
 		(dnp no)
-		(property "Reference" "C1"
+		(property "Reference" "C8"
 			(at 111.9632 68.6816 0)
 			(effects
@@
 			)
 		)
-		(property "Footprint" "custom:C_0603_1608Metric"
+		(property "Footprint" "Capacitor_SMD:C_0603_1608Metric"
 			(at 114.3 69.85 0)
 			(effects
@@
 			(project "watch"
 				(path "/71c31975-2c45-4d18-a25a-18e07a55d11e/53708456-0ae3-4e95-bf36-829cd83d6b3b"
-					(reference "C1")
+					(reference "C8")
 					(unit 1)
 				)
@@
 		(on_board yes)
 		(dnp no)
-		(property "Reference" "R1"
+		(property "Reference" "R8"
 			(at 187.452 55.88 0)
 			(effects
@@
 			)
 		)
-		(property "Footprint" "custom:R_0603_1608Metric"
+		(property "Footprint" "Resistor_SMD:R_0603_1608Metric_Pad0.98x0.95mm_HandSolder"
 			(at 184.15 54.61 0)
 			(effects
@@
 			(project "watch"
 				(path "/71c31975-2c45-4d18-a25a-18e07a55d11e/53708456-0ae3-4e95-bf36-829cd83d6b3b"
-					(reference "R1")
+					(reference "R8")
 					(unit 1)
 				)
@@
 		(on_board yes)
 		(dnp no)
-		(property "Reference" "R3"
+		(property "Reference" "R7"
 			(at 182.626 55.9054 0)
 			(effects
@@
 			)
 		)
-		(property "Footprint" "custom:R_0603_1608Metric"
+		(property "Footprint" "Resistor_SMD:R_0603_1608Metric_Pad0.98x0.95mm_HandSolder"
 			(at 179.07 54.61 0)
 			(effects
@@
 			(project "watch"
 				(path "/71c31975-2c45-4d18-a25a-18e07a55d11e/53708456-0ae3-4e95-bf36-829cd83d6b3b"
-					(reference "R3")
-					(unit 1)
-				)
+					(reference "R7")
+					(unit 1)
+				)

Commit message: review
Parts:
- R6, R7: value 2k -> 47K
- R8: value 10K -> 1M
Changed lines of the file:
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@@
 			)
 		)
-		(property "Value" "2k"
+		(property "Value" "47K"
 			(at 177.8 53.594 0)
 			(effects
@@
 			)
 		)
-		(property "Value" "10K"
+		(property "Value" "1M"
 			(at 187.452 53.594 0)
 			(effects
@@
 			)
 		)
-		(property "Value" "2k"
+		(property "Value" "47K"
 			(at 182.626 53.594 0)
 			(effects

Commit message: PCB V2
Parts:
- renumbered C8 to C11, C9 to C12, C10 to C13
Changed lines of the file:
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@@
 		(on_board yes)
 		(dnp no)
-		(property "Reference" "C9"
+		(property "Reference" "C12"
 			(at 122.1232 68.6816 0)
 			(effects
@@
 			(project "watch"
 				(path "/71c31975-2c45-4d18-a25a-18e07a55d11e/53708456-0ae3-4e95-bf36-829cd83d6b3b"
-					(reference "C9")
+					(reference "C12")
 					(unit 1)
 				)
@@
 		(on_board yes)
 		(dnp no)
-		(property "Reference" "C10"
+		(property "Reference" "C13"
 			(at 132.2832 68.6816 0)
 			(effects
@@
 			(project "watch"
 				(path "/71c31975-2c45-4d18-a25a-18e07a55d11e/53708456-0ae3-4e95-bf36-829cd83d6b3b"
-					(reference "C10")
+					(reference "C13")
 					(unit 1)
 				)
@@
 		(on_board yes)
 		(dnp no)
-		(property "Reference" "C8"
+		(property "Reference" "C11"
 			(at 111.9632 68.6816 0)
 			(effects
@@
 			(project "watch"
 				(path "/71c31975-2c45-4d18-a25a-18e07a55d11e/53708456-0ae3-4e95-bf36-829cd83d6b3b"
-					(reference "C8")
-					(unit 1)
-				)
+					(reference "C11")
+					(unit 1)
+				)
