File: watch.kicad_sch (KiCad schematic)
At the start: 17 parts, among them U2 STM32L071CBTx, Y2 CR_32kHz

Commit message: V2 PCB first draft
Parts:
- added C1, C13: 100nF, Capacitor_SMD:C_0603_1608Metric, symbol Device:C_Small
- added R4: 10M, Resistor_SMD:R_0603_1608Metric_Pad0.98x0.95mm_HandSolder, symbol Device:R_Small
- C2: renamed from C18; footprint custom:C_0603_1608Metric -> Capacitor_SMD:C_0603_1608Metric
- C3: renamed from C13; footprint custom:C_0603_1608Metric -> Capacitor_SMD:C_0603_1608Metric
- C4: renamed from C14; footprint custom:C_0603_1608Metric -> Capacitor_SMD:C_0603_1608Metric
- C5: renamed from C15; footprint custom:C_0603_1608Metric -> Capacitor_SMD:C_0603_1608Metric
- C6: renamed from C11; footprint custom:C_0603_1608Metric -> Capacitor_SMD:C_0603_1608Metric
- C7: renamed from C12; footprint custom:C_0603_1608Metric -> Capacitor_SMD:C_0603_1608Metric
- R1: renamed from R18; footprint custom:R_0603_1608Metric -> Resistor_SMD:R_0603_1608Metric_Pad0.98x0.95mm_HandSolder
- R2: renamed from R19; footprint custom:R_0603_1608Metric -> Resistor_SMD:R_0603_1608Metric_Pad0.98x0.95mm_HandSolder
- R3: renamed from R20; footprint custom:R_0603_1608Metric -> Resistor_SMD:R_0603_1608Metric_Pad0.98x0.95mm_HandSolder
- R5: renamed from R21; footprint custom:R_0603_1608Metric -> Resistor_SMD:R_0603_1608Metric_Pad0.98x0.95mm_HandSolder
- TP1: renamed from TP6; footprint TestPoint:TestPoint_Pad_D2.0mm -> TestPoint:TestPoint_Pad_D1.0mm
- TP2: renamed from TP7; footprint TestPoint:TestPoint_Pad_D2.0mm -> TestPoint:TestPoint_Pad_D1.0mm
- TP3: renamed from TP8; footprint TestPoint:TestPoint_Pad_D2.0mm -> TestPoint:TestPoint_Pad_D1.0mm
- TP4: renamed from TP9; footprint TestPoint:TestPoint_Pad_D2.0mm -> TestPoint:TestPoint_Pad_D1.0mm
- TP5: renamed from TP10; footprint TestPoint:TestPoint_Pad_D2.0mm -> TestPoint:TestPoint_Pad_D1.0mm
- renumbered U2 to U1, Y2 to Y1
Connections:
- net +BATT: now also R4.2
- net GND: now also U1.23 (VSS), U1.35 (VSS), U1.47 (VSS), U1.8 (VSSA), C1.2, C13.1
- net VDD: now also C13.2; no longer U1.23 (VSS), U1.35 (VSS), U1.47 (VSS), U1.8 (VSSA)
- net at U1.15 (PA5): now also C1.1, R4.1
- no-connect marks 0 -> 7

Commit message: review
Parts:
- added C14, C15: 100nF, Capacitor_SMD:C_0603_1608Metric, symbol Device:C_Small
- R4: value 10M -> 1M
- R5: value 10K -> 1M
Connections:
- net GND: now also C14.1, C15.1
- net VDD: now also C14.2, C15.2
Changed lines of the file:
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@@
 	)
 	(junction
+		(at 187.96 44.45)
+		(diameter 0)
+		(color 0 0 0 0)
+	)
+	(junction
 		(at 147.32 54.61)
 		(diameter 0)
@@
 	)
 	(junction
+		(at 177.8 54.61)
+		(diameter 0)
+		(color 0 0 0 0)
+	)
+	(junction
+		(at 177.8 44.45)
+		(diameter 0)
+		(color 0 0 0 0)
+	)
+	(junction
 		(at 119.38 146.05)
 		(diameter 0)
@@
 	)
 	(junction
+		(at 187.96 54.61)
+		(diameter 0)
+		(color 0 0 0 0)
+	)
+	(junction
 		(at 157.48 44.45)
 		(diameter 0)
@@
 	(wire
 		(pts
+			(xy 177.8 54.61) (xy 187.96 54.61)
+		)
+		(stroke
+			(width 0)
+			(type default)
+		)
+	)
+	(wire
+		(pts
 			(xy 134.62 118.11) (xy 132.08 118.11)
 		)
@@
 	(wire
 		(pts
+			(xy 132.08 113.03) (xy 158.75 113.03)
+		)
+		(stroke
+			(width 0)
+			(type default)
+		)
+	)
+	(wire
+		(pts
 			(xy 157.48 46.99) (xy 157.48 44.45)
 		)
@@
 	(wire
 		(pts
+			(xy 177.8 44.45) (xy 187.96 44.45)
+		)
+		(stroke
+			(width 0)
+			(type default)
+		)
+	)
+	(wire
+		(pts
 			(xy 171.45 134.62) (xy 175.26 134.62)
 		)
@@
 	(wire
 		(pts
-			(xy 158.75 113.03) (xy 132.08 113.03)
+			(xy 187.96 54.61) (xy 187.96 52.07)
 		)
 		(stroke
@@
 	(wire
 		(pts
+			(xy 187.96 44.45) (xy 198.12 44.45)
+		)
+		(stroke
+			(width 0)
+			(type default)
+		)
+	)
+	(wire
+		(pts
 			(xy 33.02 26.67) (xy 26.67 26.67)
 		)
@@
 	(wire
 		(pts
+			(xy 187.96 54.61) (xy 198.12 54.61)
+		)
+		(stroke
+			(width 0)
+			(type default)
+		)
+	)
+	(wire
+		(pts
 			(xy 109.22 146.05) (xy 109.22 135.89)
 		)
@@
 	(wire
 		(pts
-			(xy 134.62 125.73) (xy 134.62 120.65)
+			(xy 134.62 120.65) (xy 134.62 125.73)
 		)
 		(stroke
@@
 	(wire
 		(pts
+			(xy 198.12 44.45) (xy 198.12 46.99)
+		)
+		(stroke
+			(width 0)
+			(type default)
+		)
+	)
+	(wire
+		(pts
 			(xy 173.99 123.19) (xy 175.26 123.19)
 		)
@@
 	(wire
 		(pts
-			(xy 167.64 110.49) (xy 132.08 110.49)
+			(xy 198.12 52.07) (xy 198.12 54.61)
 		)
 		(stroke
@@
 	(wire
 		(pts
+			(xy 187.96 44.45) (xy 187.96 46.99)
+		)
+		(stroke
+			(width 0)
+			(type default)
+		)
+	)
+	(wire
+		(pts
 			(xy 66.04 90.17) (xy 66.04 93.98)
 		)
@@
 	(wire
 		(pts
+			(xy 132.08 110.49) (xy 167.64 110.49)
+		)
+		(stroke
+			(width 0)
+			(type default)
+		)
+	)
+	(wire
+		(pts
 			(xy 167.64 127) (xy 167.64 123.19)
 		)
@@
 			)
 		)
-		(property "Value" "10K"
+		(property "Value" "1M"
 			(at 146.558 120.65 90)
 			(effects
@@
 		(on_board yes)
 		(dnp no)
-		(fields_autoplaced yes)
 		(property "Reference" "U1"
 			(at 112.1059 57.15 0)
@@
 			)
 		)
-		(property "Value" "10M"
+		(property "Value" "1M"
 			(at 69.596 76.454 0)
 			(effects
@@
 					(unit 1)
 				)
+			)
+		)
+	)
+	(symbol
+		(lib_id "Device:C_Small")
+		(at 198.12 49.53 0)
+		(mirror x)
+		(unit 1)
+		(exclude_from_sim no)
+		(in_bom yes)
+		(on_board yes)
+		(dnp no)
+		(property "Reference" "C15"
+			(at 200.4568 50.6984 0)
+			(effects
+				(font
+					(size 1.27 1.27)
+				)
+				(justify left)
+			)
+		)
+		(property "Value" "100nF"
+			(at 200.4568 48.387 0)
+			(effects
+				(font
+					(size 1.27 1.27)
+				)
+				(justify left)
+			)
+		)
+		(property "Footprint" "Capacitor_SMD:C_0603_1608Metric"
+			(at 198.12 49.53 0)
+			(effects
+				(font
+					(size 1.27 1.27)
+				)
+				(hide yes)
+			)
+		)
+		(property "Datasheet" "~"
+			(at 198.12 49.53 0)
+			(effects
+				(font
+					(size 1.27 1.27)
+				)
+				(hide yes)
+			)
+		)
+		(property "Description" ""
+			(at 198.12 49.53 0)
+			(effects
+				(font
+					(size 1.27 1.27)
+				)
+				(hide yes)
+			)
+		)
+		(pin "1"
+		)
+		(pin "2"
+		)
+		(instances
+			(project "watch"
+				(path "/71c31975-2c45-4d18-a25a-18e07a55d11e"
+					(reference "C15")
+					(unit 1)
+				)
+			)
+		)
+	)
+	(symbol
+		(lib_id "Device:C_Small")
+		(at 187.96 49.53 0)
+		(mirror x)
+		(unit 1)
+		(exclude_from_sim no)
+		(in_bom yes)
+		(on_board yes)
+		(dnp no)
+		(property "Reference" "C14"
+			(at 190.2968 50.6984 0)
+			(effects
+				(font
+					(size 1.27 1.27)
+				)
+				(justify left)
+			)
+		)
+		(property "Value" "100nF"
+			(at 190.2968 48.387 0)
+			(effects
+				(font
+					(size 1.27 1.27)
+				)
+				(justify left)
+			)
+		)
+		(property "Footprint" "Capacitor_SMD:C_0603_1608Metric"
+			(at 187.96 49.53 0)
+			(effects
+				(font
+					(size 1.27 1.27)
+				)
+				(hide yes)
+			)
+		)
+		(property "Datasheet" "~"
+			(at 187.96 49.53 0)
+			(effects
+				(font
+					(size 1.27 1.27)
+				)
+				(hide yes)
+			)
+		)
+		(property "Description" ""
+			(at 187.96 49.53 0)
+			(effects
+				(font
+					(size 1.27 1.27)
+				)
+				(hide yes)
+			)
+		)
+		(pin "1"
+		)
+		(pin "2"
+		)
+		(instances
+			(project "watch"
+				(path "/71c31975-2c45-4d18-a25a-18e07a55d11e"
+					(reference "C14")
+					(unit 1)
+				)

Commit message: PCB V2
Parts:
- renumbered C15 to C10, C13 to C8, C14 to C9
Connections:
- net Power/SEL_VDD: now reaches U1.16 (PA6)
- no-connect marks 7 -> 6
Other:
- sheet Power ports: added SEL_VDD; removed none
Changed lines of the file:
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@@
 		(at 99.06 102.87)
 	)
-	(no_connect
-		(at 99.06 115.57)
-	)
 	(wire
 		(pts
@@
 	(wire
 		(pts
+			(xy 80.01 115.57) (xy 99.06 115.57)
+		)
+		(stroke
+			(width 0)
+			(type default)
+		)
+	)
+	(wire
+		(pts
 			(xy 43.18 41.91) (xy 54.61 41.91)
 		)
@@
 	(wire
 		(pts
+			(xy 80.01 59.69) (xy 46.99 59.69)
+		)
+		(stroke
+			(width 0)
+			(type default)
+		)
+	)
+	(wire
+		(pts
 			(xy 54.61 21.59) (xy 38.1 21.59)
 		)
@@
 	(wire
 		(pts
+			(xy 80.01 115.57) (xy 80.01 59.69)
+		)
+		(stroke
+			(width 0)
+			(type default)
+		)
+	)
+	(wire
+		(pts
 			(xy 134.62 133.35) (xy 134.62 130.81)
 		)
@@
 		(on_board yes)
 		(dnp no)
-		(property "Reference" "C15"
+		(property "Reference" "C10"
 			(at 200.4568 50.6984 0)
 			(effects
@@
 			(project "watch"
 				(path "/71c31975-2c45-4d18-a25a-18e07a55d11e"
-					(reference "C15")
+					(reference "C10")
 					(unit 1)
 				)
@@
 		(on_board yes)
 		(dnp no)
-		(property "Reference" "C14"
+		(property "Reference" "C9"
 			(at 190.2968 50.6984 0)
 			(effects
@@
 			(project "watch"
 				(path "/71c31975-2c45-4d18-a25a-18e07a55d11e"
-					(reference "C14")
+					(reference "C9")
 					(unit 1)
 				)
@@
 		(on_board yes)
 		(dnp no)
-		(property "Reference" "C13"
+		(property "Reference" "C8"
 			(at 180.1368 50.6984 0)
 			(effects
@@
 			(project "watch"
 				(path "/71c31975-2c45-4d18-a25a-18e07a55d11e"
-					(reference "C13")
+					(reference "C8")
 					(unit 1)
 				)
@@
 			)
 		)
+		(pin "SEL_VDD" input
+			(at 46.99 59.69 0)
+			(effects
+				(font
+					(size 1.27 1.27)
+				)
+				(justify right)
+			)
+		)
