File: watch.kicad_sch (KiCad schematic)
At the start: 91 parts, among them U1 STM32L071CBTx, U2 BOSCH BMA400, Y1 3131M-32.768DTTLRRL

Commit message: removed old project files
Parts:
- BT1: now left out of the parts list
- C7, C8: LCSC Part # C326779 -> C527046
Connections:
- net IMU_SCL: now also R2.2, U2.12 (SCL); no longer R1.2, U2.2 (SDA)
- net IMU_SDA: now also R1.2, U2.2 (SDA); no longer R2.2, U2.12 (SCL)
- net VDD: no longer U1.17 (PA7)
- no-connect marks 12 -> 13
Other:
- moved on the sheet: R10, R8, R9, TP1, TP2, TP3, TP4, TP5
