File: power.kicad_sch (KiCad schematic)
At the start: 8 parts, among them U4 TPS63900

Commit message: V2 PCB first draft
Parts:
- BT1: renamed from BT2; footprint SamacSys_Parts:BATHLD001 -> custom_lib:BatteryHolder_CR2016
- C11: renamed from C16; footprint (none) -> Capacitor_SMD:C_0603_1608Metric
- C12: renamed from C17; footprint (none) -> Capacitor_SMD:C_0603_1608Metric
- L1: renamed from L2; footprint (none) -> Inductor_SMD:L_0603_1608Metric_Pad1.05x0.95mm_HandSolder
- R21: renamed from R24; footprint custom:R_0603_1608Metric -> Resistor_SMD:R_0603_1608Metric_Pad0.98x0.95mm_HandSolder
- R22: renamed from R25; footprint custom:R_0603_1608Metric -> Resistor_SMD:R_0603_1608Metric_Pad0.98x0.95mm_HandSolder
- R23: renamed from R26; footprint custom:R_0603_1608Metric -> Resistor_SMD:R_0603_1608Metric_Pad0.98x0.95mm_HandSolder
- renumbered U4 to U3
Changed lines of the file:
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@@
 		(dnp no)
 		(fields_autoplaced yes)
-		(property "Reference" "#PWR040"
+		(property "Reference" "#PWR025"
 			(at 138.43 54.61 0)
 			(effects
@@
 			(project "watch"
 				(path "/71c31975-2c45-4d18-a25a-18e07a55d11e/c88e79a5-24fb-4b9a-9b6f-dfb9921812a0"
-					(reference "#PWR040")
+					(reference "#PWR025")
 					(unit 1)
 				)
@@
 		(on_board yes)
 		(dnp no)
-		(property "Reference" "R25"
+		(property "Reference" "R22"
 			(at 128.27 77.47 90)
 			(effects
@@
 			)
 		)
-		(property "Footprint" "custom:R_0603_1608Metric"
+		(property "Footprint" "Resistor_SMD:R_0603_1608Metric_Pad0.98x0.95mm_HandSolder"
 			(at 125.73 74.93 0)
 			(effects
@@
 			(project "watch"
 				(path "/71c31975-2c45-4d18-a25a-18e07a55d11e/c88e79a5-24fb-4b9a-9b6f-dfb9921812a0"
-					(reference "R25")
+					(reference "R22")
 					(unit 1)
 				)
@@
 		(dnp no)
 		(fields_autoplaced yes)
-		(property "Reference" "L2"
+		(property "Reference" "L1"
 			(at 91.44 68.5799 0)
 			(effects
@@
 			)
 		)
-		(property "Footprint" ""
+		(property "Footprint" "Inductor_SMD:L_0603_1608Metric_Pad1.05x0.95mm_HandSolder"
 			(at 90.17 69.85 0)
 			(effects
@@
 			(project "watch"
 				(path "/71c31975-2c45-4d18-a25a-18e07a55d11e/c88e79a5-24fb-4b9a-9b6f-dfb9921812a0"
-					(reference "L2")
+					(reference "L1")
 					(unit 1)
 				)
@@
 		(on_board yes)
 		(dnp no)
-		(property "Reference" "R24"
+		(property "Reference" "R21"
 			(at 123.19 77.47 90)
 			(effects
@@
 			)
 		)
-		(property "Footprint" "custom:R_0603_1608Metric"
+		(property "Footprint" "Resistor_SMD:R_0603_1608Metric_Pad0.98x0.95mm_HandSolder"
 			(at 120.65 74.93 0)
 			(effects
@@
 			(project "watch"
 				(path "/71c31975-2c45-4d18-a25a-18e07a55d11e/c88e79a5-24fb-4b9a-9b6f-dfb9921812a0"
-					(reference "R24")
+					(reference "R21")
 					(unit 1)
 				)
@@
 		(on_board yes)
 		(dnp no)
-		(property "Reference" "BT2"
+		(property "Reference" "BT1"
 			(at 49.784 61.468 0)
 			(effects
@@
 			)
 		)
-		(property "Footprint" "SamacSys_Parts:BATHLD001"
+		(property "Footprint" "custom_lib:BatteryHolder_CR2016"
 			(at 68.58 59.436 90)
 			(effects
@@
 			(project "watch"
 				(path "/71c31975-2c45-4d18-a25a-18e07a55d11e/c88e79a5-24fb-4b9a-9b6f-dfb9921812a0"
-					(reference "BT2")
+					(reference "BT1")
 					(unit 1)
 				)
@@
 		(on_board yes)
 		(dnp no)
-		(property "Reference" "#PWR039"
+		(property "Reference" "#PWR024"
 			(at 106.68 91.44 0)
 			(effects
@@
 			(project "watch"
 				(path "/71c31975-2c45-4d18-a25a-18e07a55d11e/c88e79a5-24fb-4b9a-9b6f-dfb9921812a0"
-					(reference "#PWR039")
+					(reference "#PWR024")
 					(unit 1)
 				)
@@
 		(dnp no)
 		(fields_autoplaced yes)
-		(property "Reference" "#PWR042"
+		(property "Reference" "#PWR023"
 			(at 68.58 54.61 0)
 			(effects
@@
 			(project "watch"
 				(path "/71c31975-2c45-4d18-a25a-18e07a55d11e/c88e79a5-24fb-4b9a-9b6f-dfb9921812a0"
-					(reference "#PWR042")
+					(reference "#PWR023")
 					(unit 1)
 				)
@@
 		(dnp no)
 		(fields_autoplaced yes)
-		(property "Reference" "U4"
+		(property "Reference" "U3"
 			(at 106.68 46.99 0)
 			(effects
@@
 			(project "watch"
 				(path "/71c31975-2c45-4d18-a25a-18e07a55d11e/c88e79a5-24fb-4b9a-9b6f-dfb9921812a0"
-					(reference "U4")
+					(reference "U3")
 					(unit 1)
 				)
@@
 		(dnp no)
 		(fields_autoplaced yes)
-		(property "Reference" "C16"
+		(property "Reference" "C11"
 			(at 80.01 58.4262 0)
 			(effects
@@
 			)
 		)
-		(property "Footprint" ""
+		(property "Footprint" "Capacitor_SMD:C_0603_1608Metric"
 			(at 77.47 59.69 0)
 			(effects
@@
 			(project "watch"
 				(path "/71c31975-2c45-4d18-a25a-18e07a55d11e/c88e79a5-24fb-4b9a-9b6f-dfb9921812a0"
-					(reference "C16")
+					(reference "C11")
 					(unit 1)
 				)
@@
 		(on_board yes)
 		(dnp no)
-		(property "Reference" "R26"
+		(property "Reference" "R23"
 			(at 133.35 77.47 90)
 			(effects
@@
 			)
 		)
-		(property "Footprint" "custom:R_0603_1608Metric"
+		(property "Footprint" "Resistor_SMD:R_0603_1608Metric_Pad0.98x0.95mm_HandSolder"
 			(at 130.81 74.93 0)
 			(effects
@@
 			(project "watch"
 				(path "/71c31975-2c45-4d18-a25a-18e07a55d11e/c88e79a5-24fb-4b9a-9b6f-dfb9921812a0"
-					(reference "R26")
+					(reference "R23")
 					(unit 1)
 				)
@@
 		(dnp no)
 		(fields_autoplaced yes)
-		(property "Reference" "C17"
+		(property "Reference" "C12"
 			(at 140.97 59.6962 0)
 			(effects
@@
 			)
 		)
-		(property "Footprint" ""
+		(property "Footprint" "Capacitor_SMD:C_0603_1608Metric"
 			(at 138.43 60.96 0)
 			(effects
@@
 			(project "watch"
 				(path "/71c31975-2c45-4d18-a25a-18e07a55d11e/c88e79a5-24fb-4b9a-9b6f-dfb9921812a0"
-					(reference "C17")
-					(unit 1)
-				)
+					(reference "C12")
+					(unit 1)
+				)

Commit message: review
Parts:
- added R24: 560K, Resistor_SMD:R_0603_1608Metric_Pad0.98x0.95mm_HandSolder, symbol Device:R_Small
- added R25: 1K8, Resistor_SMD:R_0603_1608Metric_Pad0.98x0.95mm_HandSolder, symbol Device:R_Small
- added R26: 15K, Resistor_SMD:R_0603_1608Metric_Pad0.98x0.95mm_HandSolder, symbol Device:R_Small
- R21: value 16.2K -> 1K2
- R22: value 1.87K -> 68
- R23: value 36.5K -> 39K
Connections:
- net GND: now also R24.1, R25.1, R26.1; no longer R21.1, R22.1
- net at R23.2, U3.3 (CFG1): now also R24.2
- new net: R22.1, R25.2
- new net: R21.1, R26.2
Other:
- moved on the sheet: C12, R23

Commit message: PCB V2
Parts:
- removed R21: 1K2, Resistor_SMD:R_0603_1608Metric_Pad0.98x0.95mm_HandSolder, symbol Device:R_Small
- removed R26: 15K, Resistor_SMD:R_0603_1608Metric_Pad0.98x0.95mm_HandSolder, symbol Device:R_Small
- added R21: 10K, Resistor_SMD:R_0603_1608Metric_Pad0.98x0.95mm_HandSolder, symbol Device:R
- added R22: 1M, Resistor_SMD:R_0603_1608Metric_Pad0.98x0.95mm_HandSolder, symbol Device:R
- renumbered C11 to C14, C12 to C15, R22 to R23, R25 to R24, R23 to R25, R24 to R26
Connections:
- net +BATT: no longer U3.2 (SEL)
- net GND: now also U3.5 (CFG3), R22.2
- new net: R21.2, R22.1, U3.2 (SEL)
- new net SEL_VDD: R21.1
Other:
- moved on the sheet: BT1, C14

Commit message: small fixes
Parts:
- added R27: 510, Resistor_SMD:R_0603_1608Metric_Pad0.98x0.95mm_HandSolder, symbol Device:R_Small
Connections:
- net GND: now also R27.1; no longer U3.5 (CFG3)
- new net: R27.2, U3.5 (CFG3)
Changed lines of the file:
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@@
+	(wire
+		(pts
+			(xy 120.65 88.9) (xy 120.65 95.25)
+		)
+		(stroke
+			(width 0)
+			(type default)
+		)
+	)
 	(wire
 		(pts
@@
 	(wire
 		(pts
+			(xy 116.84 54.61) (xy 142.24 54.61)
+		)
+		(stroke
+			(width 0)
+			(type default)
+		)
+	)
+	(wire
+		(pts
 			(xy 77.47 62.23) (xy 81.28 62.23)
 		)
@@
 	(wire
 		(pts
-			(xy 120.65 69.85) (xy 120.65 95.25)
+			(xy 120.65 69.85) (xy 120.65 83.82)
 		)
 		(stroke
@@
 		(pts
 			(xy 135.89 91.44) (xy 135.89 95.25)
-		)
-		(stroke
-			(width 0)
-			(type default)
-		)
-	)
-	(wire
-		(pts
-			(xy 116.84 54.61) (xy 142.24 54.61)
 		)
 		(stroke
@@
 					(unit 1)
 				)
+			)
+		)
+	)
+	(symbol
+		(lib_id "Device:R_Small")
+		(at 120.65 86.36 180)
+		(unit 1)
+		(exclude_from_sim no)
+		(in_bom yes)
+		(on_board yes)
+		(dnp no)
+		(property "Reference" "R27"
+			(at 123.19 88.9 90)
+			(effects
+				(font
+					(size 1.27 1.27)
+				)
+			)
+		)
+		(property "Value" "510"
+			(at 123.19 83.82 90)
+			(effects
+				(font
+					(size 1.27 1.27)
+				)
+			)
+		)
+		(property "Footprint" "Resistor_SMD:R_0603_1608Metric_Pad0.98x0.95mm_HandSolder"
+			(at 120.65 86.36 0)
+			(effects
+				(font
+					(size 1.27 1.27)
+				)
+				(hide yes)
+			)
+		)
+		(property "Datasheet" "~"
+			(at 120.65 86.36 0)
+			(effects
+				(font
+					(size 1.27 1.27)
+				)
+				(hide yes)
+			)
+		)
+		(property "Description" ""
+			(at 120.65 86.36 0)
+			(effects
+				(font
+					(size 1.27 1.27)
+				)
+				(hide yes)
+			)
+		)
+		(pin "1"
+		)
+		(pin "2"
+		)
+		(instances
+			(project "watch"
+				(path "/71c31975-2c45-4d18-a25a-18e07a55d11e/c88e79a5-24fb-4b9a-9b6f-dfb9921812a0"
+					(reference "R27")
+					(unit 1)
+				)
