File: watch.kicad_pcb (KiCad board)
At the start: 2 copper layers, 38 x 38 mm, 91 parts, among them U1 STM32L071CBTx, U2 BOSCH BMA400, Y1 3131M-32.768DTTLRRL

Commit message: removed old project files
Parts:
- moved R1 1.51 mm to (56.3, 61.0)
- moved R2 1.51 mm to (55.3, 62.1)
Connections:
- R1 pad 2: IMU_SCL -> IMU_SDA
- R2 pad 2: IMU_SDA -> IMU_SCL
- U1 pad 17: VDD -> unconnected-(U1-PA7-Pad17)
- U2 pad 12: IMU_SDA -> IMU_SCL
- U2 pad 2: IMU_SCL -> IMU_SDA
Routing:
- net VDD: track 133.7 -> 114.1 mm, vias 13 -> 10
- net IMU_SCL: track 8.64 -> 11.2 mm
- net IMU_SDA: track 11.6 -> 9.13 mm
- net GND: track 82.1 -> 81.5 mm
